File: Power_Supply.sch (KiCad schematic (older format))
At the start: 12 parts, among them J201 B4B-PH-K-S_LF__SN_, U201 LM78L12_SO8, U202 LT1763CS8-5, U203 LT1763CS8-3.3

Commit message: v1.0.0
Parts:
- added H201, H202, H203, H204: MountingHole_Pad, MountingHole:MountingHole_3.2mm_M3_Pad_Via, symbol Mechanical:MountingHole_Pad
- added J202, J203: B2B-PH-K-S_LF__SN_, digikey-footprints:PinHeader_1x2_P2mm_Drill1mm, symbol dk_Rectangular-Connectors-Headers-Male-Pins:B2B-PH-K-S_LF__SN_
Connections:
- net +3V3: now also J202.1
- net +5V: now also J203.1
- net GND: now also H201.1, H202.1, H203.1, H204.1, J202.2, J203.2
Other:
- moved on the sheet: C204, C207, C208, U203
