File: Sort and Save Scanner.kicad_pcb (KiCad board)
At the start: 4 copper layers, 132.1 x 86.4 mm, 60 parts, among them J201 B4B-PH-K-S_LF__SN_, J301 FTSH-105-01-F-DV-K, J302 FTSH-105-01-F-DV-K, J401 67996-412HLF, U201 LM78L12_SO8, U202 LT1763CS8-5, U203 LT1763CS8-3.3, U301 STM32F051R8Tx, U401 OPA2376AIDR-8, U402 REF5025AD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

Commit message: v1.0.0
Parts:
- added H201: MountingHole_Pad, MountingHole:MountingHole_3.2mm_M3_Pad_Via, F.Cu at (119.4, 128.3)
- added H202: MountingHole_Pad, MountingHole:MountingHole_3.2mm_M3_Pad_Via, F.Cu at (119.4, 166.4)
- added H203: MountingHole_Pad, MountingHole:MountingHole_3.2mm_M3_Pad_Via, F.Cu at (154.9, 128.3)
- added H204: MountingHole_Pad, MountingHole:MountingHole_3.2mm_M3_Pad_Via, F.Cu at (154.9, 166.4)
- added H301: MountingHole_Pad, MountingHole:MountingHole_3.2mm_M3_Pad_Via, F.Cu at (78.7, 68.6)
- added H302: MountingHole_Pad, MountingHole:MountingHole_3.2mm_M3_Pad_Via, F.Cu at (78.7, 106.7)
- added H303: MountingHole_Pad, MountingHole:MountingHole_3.2mm_M3_Pad_Via, F.Cu at (114.3, 68.6)
- added H304: MountingHole_Pad, MountingHole:MountingHole_3.2mm_M3_Pad_Via, F.Cu at (114.3, 106.7)
- added J202: B2B-PH-K-S_LF__SN_, digikey-footprints:PinHeader_1x2_P2mm_Drill1mm, F.Cu at (127.0, 147.3)
- added J203: B2B-PH-K-S_LF__SN_, digikey-footprints:PinHeader_1x2_P2mm_Drill1mm, F.Cu at (127.0, 154.9)
- added J303: B4B-PH-K-S_LF__SN_, digikey-footprints:PinHeader_1x4_P2mm_Drill1mm, F.Cu at (80.0, 97.8)
- added J304: B2B-PH-K-S_LF__SN_, digikey-footprints:PinHeader_1x2_P2mm_Drill1mm, F.Cu at (105.4, 74.9)
- D405: footprint LED_SMD:LED_0603_1608Metric -> LED_SMD:LED_1206_3216Metric
- D406: value 950nm -> 940nm; footprint LED_SMD:LED_0402_1005Metric -> LED_SMD:LED_1206_3216Metric
- R402: value 39 -> 66
- moved C201 13.1 mm to (133.3, 142.2)
- moved C205 13.1 mm to (132.1, 156.2)
- moved C207 13.1 mm to (132.1, 148.6)
- moved U201 13.1 mm to (138.4, 141.0)
- moved U203 13.1 mm to (138.4, 148.6)
- moved C206 13.1 mm to (133.3, 156.2)
- moved C208 13.1 mm to (133.3, 148.6)
- moved J201 13.1 mm to (135.7, 134.6)
- moved U202 13.1 mm to (138.6, 156.2)
- moved C202 13.1 mm to (143.5, 142.2)
- moved C203 13.1 mm to (143.5, 154.9)
- moved C204 13.1 mm to (143.5, 147.3)
- moved D405 9.67 mm to (181.6, 80.0)
- moved C402 9.25 mm to (165.1, 99.1)
- moved C403 9.25 mm to (175.3, 99.1)
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Connections:
- J401 pad 1: Net-(J401-Pad1) -> GND
Routing:
- net GND: track 142.7 -> 201.6 mm, vias 25 -> 38
- net +3V3: track 63.3 -> 76.6 mm, vias 3 -> 5
- net /ARM Board/UART_TX: track 0.00 -> 13.2 mm, vias 0 -> 1
- net /ARM Board/UART_RX: track 0.00 -> 11.9 mm, vias 0 -> 1
- net +5V: track 16.8 -> 22.2 mm
- net Net-(J301-Pad9): track 1.68 -> 3.23 mm
- net Net-(D405-Pad1): track 2.10 -> 3.45 mm
- net /Sensor/LED_PWR_IN5: track 27.0 -> 27.8 mm
- net /Sensor/LED_PWR_IN7: track 22.4 -> 22.0 mm, vias 0 -> 2
Other:
- board size 132.1 x 86.4 mm -> 127 x 107.9 mm

Commit message: v1.0.0
Parts:
- moved D405 1.27 mm to (181.6, 78.7)
- moved R401 1.27 mm to (181.6, 76.2)
Routing:
- net GND: track 201.6 -> 202.1 mm
- net /Sensor/LED_PWR_IN8: track 35.6 -> 36.1 mm
Other:
- outline, holes or cut-outs redrawn

Commit message: v1.0.0
Parts:
- moved C401 1.25 mm to (198.0, 101.2), turned to 270 degrees
- moved C405 0.83 mm to (196.7, 101.2), turned to 90 degrees
- moved J303 0.19 mm to (80.0, 98.0)
Routing:
- net GND: track 202.1 -> 91.1 mm, vias 38 -> 30
- net +3V3: track 76.6 -> 63.5 mm, vias 5 -> 4
- net +5V: track 22.2 -> 17.1 mm, vias 3 -> 2
- net /ARM Board/HSE_IN: track 10.3 -> 8.57 mm
- net /Sensor/LED_PWR_IN1: track 37.5 -> 38.6 mm
Other:
- net class Default: via_dia 0.8 -> 0.4; via_drill 0.4 -> 0.2
- rule trace_min: 0.15 -> 0.077
- rule via_min_drill: 0.3 -> 0.16
